File: BLDC_Cont.sch (KiCad schematic (older format))
At the start: 24 parts, among them J1 Conn, J2 Conn, J3 Conn, J4 Conn_01x05_Female, J5 Conn_01x02_Female, Q1 BUK9Y14-80E, Q2 BUK9Y14-80E, U1 ADUM7234

Commit message: Rev. 3
Updated Revision (3)
-Organized files
-Removed legacy documentation
-Found cross-conduction protection of ADuM7234 was **NOT** satisfactory.
+Added NOR gate based mutual exclusion circuit.
Parts:
- added C8: 1 uF, Capacitor_SMD:C_1206_3216Metric_Pad1.33x1.80mm_HandSolder, symbol Device:C_Small
- added C9: 0.1 uF, Capacitor_SMD:C_1206_3216Metric_Pad1.33x1.80mm_HandSolder, symbol Device:C_Small
- added J6: Pin Headder, Connector_PinHeader_2.54mm:PinHeader_1x02_P2.54mm_Vertical, symbol Connector:Conn_01x02_Female
- added U2: 74HC7002, Package_SO:SOIC-14_3.9x8.7mm_P1.27mm, symbol 74hc7002:74HC7002
- J4: value Conn_01x05_Female -> Pin Headder; footprint Connector_PinHeader_2.54mm:PinHeader_1x05_P2.54mm_Vertical -> Connector_PinHeader_2.54mm:PinHeader_1x04_P2.54mm_Vertical; symbol Connector:Conn_01x05_Female -> Connector:Conn_01x04_Female
- J5: value Conn_01x02_Female -> GND_Jumper
Connections:
- net +12V: now also J6.1 (Pin_1); no longer J4.1 (Pin_1)
- net +5VD: now also J4.1 (Pin_1), C8.1, C9.1, U2.14 (VCC); no longer J4.4 (Pin_4)
- net GNDD: now also J4.4 (Pin_4), C8.2, C9.2, U2.2, U2.5, U2.7 (GND); no longer J4.5 (Pin_5)
- net PWM_A: now also U2.1, U2.10; no longer U1.2 (V_IA)
- net PWM_B: now also U2.12, U2.4; no longer U1.3 (V_IB)
- net GND renamed GNDPWR
- net GNDPWR: now also J6.2 (Pin_2)
- new net A_Safe: U1.2 (V_IA), U2.11
- new net B_Safe: U1.3 (V_IB), U2.8
- new net nA: U2.13, U2.3
- new net nB: U2.6, U2.9
Other:
- moved on the sheet: C1, C2, C3, C4, C5, C6, C7, D1, D2, D3, D4, J1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
